File: KiCAD/projet-capteur/projet-capteur.kicad_pcb (KiCad board)
At the start: 2 copper layers, 75.5 x 65.8 mm, 25 parts, among them J1 Power, J2 Analog, J3 Digital/PWM, J4 Digital/PWM, U2 LTC1050

Commit message: Modif Rot
Parts:
- removed MH1, MH2, MH3, MH4: MountingHole_3.2mm, Arduino_MountingHole:MountingHole_3.2mm
- moved ROE1 22.1 mm to (168.5, 57.0), turned to 90 degrees
- moved CG1 2.20 mm to (124.5, 70.0)
- moved U1 2.00 mm to (159.0, 80.5)
- moved C4 1.12 mm to (168.5, 42.5), turned to -90 degrees
Routing:
- net ROE 3: track 6.69 -> 24.0 mm
- net ROE 4: track 5.50 -> 17.9 mm
- net /*11: track 32.1 -> 29.1 mm
- net ROE 5: track 13.6 -> 16.0 mm
- net R3: track 38.8 -> 40.3 mm
- net SCL: track 16.7 -> 17.7 mm
- net Out Sensor: track 5.03 -> 5.94 mm
- net SDA: track 13.1 -> 14.0 mm
