File: KiCAD/projet-capteur/projet-capteur.kicad_pcb (KiCad board)
At the start: 2 copper layers, 75.5 x 65.8 mm, 21 parts, among them J1 Power, J2 Analog, J3 Digital/PWM, J4 Digital/PWM, U2 LTC1050

Commit message: Beautification du PCB
Parts:
- moved R6 53.2 mm to (104.5, 97.6), turned to 90 degrees
- moved FS1 42.0 mm to (110.4, 96.2), turned to 90 degrees
- moved U3 30.9 mm to (106.2, 49.2)
- moved R1 24.7 mm to (102.0, 76.2), turned to 0 degrees
- moved CG1 22.5 mm to (102.0, 69.7)
- moved C3 9.55 mm to (150.8, 91.2), turned to 180 degrees
- moved C2 1.86 mm to (141.1, 81.6)
- moved R4 1.79 mm to (136.0, 81.5)
- moved R5 0.17 mm to (145.7, 86.6), turned to 0 degrees
Connections:
- J3 pad 10: TX -> RX
- J4 pad 1: RX -> TX
Routing:
- net 5V: track 205.3 -> 259.1 mm
- net Out Flex: track 8.58 -> 52.5 mm
- net TX: track 8.81 -> 51.0 mm
- net RX: track 9.65 -> 44.8 mm
- net ADC: track 19.9 -> 10.9 mm
- net /AO+: track 15.3 -> 23.2 mm
- net /AO Out: track 39.1 -> 38.4 mm
- net Out Sensor: track 5.94 -> 5.25 mm
Other:
- board text removed: "ICSP"

Commit message: Beautification du Schematique
Connections:
- net /*10 renamed CS Pot
- net /*11 renamed SDI Pot
- net /*9 renamed DATA Serv
- net /13 renamed SCK Pot
Changed lines of the file:
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@@
 	(net 9 "SDA")
 	(net 10 "/12")
-	(net 11 "/13")
+	(net 11 "SDI Pot")
 	(net 12 "/AREF")
-	(net 13 "/*11")
-	(net 14 "/*10")
-	(net 15 "/*9")
+	(net 13 "SCK Pot")
+	(net 14 "CS Pot")
+	(net 15 "DATA Serv")
 	(net 16 "/TX{slash}1")
 	(net 17 "/RX{slash}0")
@@
 			(layers "*.Cu" "*.Mask")
 			(remove_unused_layers no)
-			(net 11 "/13")
+			(net 13 "SCK Pot")
 			(pinfunction "Pin_5")
 			(pintype "passive")
@@
 			(layers "*.Cu" "*.Mask")
 			(remove_unused_layers no)
-			(net 13 "/*11")
+			(net 11 "SDI Pot")
 			(pinfunction "Pin_7")
 			(pintype "passive")
@@
 			(layers "*.Cu" "*.Mask")
 			(remove_unused_layers no)
-			(net 14 "/*10")
+			(net 14 "CS Pot")
 			(pinfunction "Pin_8")
 			(pintype "passive")
@@
 			(layers "*.Cu" "*.Mask")
 			(remove_unused_layers no)
-			(net 15 "/*9")
+			(net 15 "DATA Serv")
 			(pinfunction "Pin_9")
 			(pintype "passive")
@@
 			(layers "*.Cu" "*.Mask")
 			(remove_unused_layers no)
-			(net 15 "/*9")
+			(net 15 "DATA Serv")
 			(pinfunction "Data")
 			(pintype "input")
@@
 			(layers "*.Cu" "*.Mask")
 			(remove_unused_layers no)
-			(net 14 "/*10")
+			(net 14 "CS Pot")
 			(pinfunction "CS")
 			(pintype "input")
@@
 			(layers "*.Cu" "*.Mask")
 			(remove_unused_layers no)
-			(net 11 "/13")
+			(net 13 "SCK Pot")
 			(pinfunction "SCK")
 			(pintype "input")
@@
 			(layers "*.Cu" "*.Mask")
 			(remove_unused_layers no)
-			(net 13 "/*11")
+			(net 11 "SDI Pot")
 			(pinfunction "SDI")
 			(pintype "input")
@@
 	)
 	(segment
-		(start 120.812922 55.590078)
-		(end 119.77 56.633)
+		(start 132.885 47.099)
+		(end 117.5 47.099)
 		(width 0.5)
 		(layer "B.Cu")
@@
 	)
 	(segment
-		(start 119.77 56.633)
-		(end 119.77 57.695)
+		(start 117.23 55.945)
+		(end 116 54.715)
 		(width 0.5)
 		(layer "B.Cu")
@@
 	)
 	(segment
-		(start 122.690078 55.590078)
-		(end 120.812922 55.590078)
+		(start 116 54.715)
+		(end 116 48)
 		(width 0.5)
 		(layer "B.Cu")
@@
 	)
 	(segment
-		(start 128.956 49.324156)
-		(end 122.690078 55.590078)
+		(start 116.901 47.099)
+		(end 117.5 47.099)
 		(width 0.5)
 		(layer "B.Cu")
@@
 	)
 	(segment
-		(start 132.885 47.099)
-		(end 117.5 47.099)
+		(start 116 48)
+		(end 116.901 47.099)
 		(width 0.5)
 		(layer "B.Cu")
-		(net 13)
+		(net 11)
 	)
 	(segment
-		(start 117.23 55.945)
-		(end 116 54.715)
+		(start 117.23 57.695)
+		(end 117.23 55.945)
 		(width 0.5)
 		(layer "B.Cu")
-		(net 13)
+		(net 11)
 	)
 	(segment
-		(start 116 54.715)
-		(end 116 48)
+		(start 134.036 48.25)
+		(end 132.885 47.099)
 		(width 0.5)
 		(layer "B.Cu")
-		(net 13)
+		(net 11)
 	)
 	(segment
-		(start 116.901 47.099)
-		(end 117.5 47.099)
+		(start 120.812922 55.590078)
+		(end 119.77 56.633)
 		(width 0.5)
 		(layer "B.Cu")
@@
 	)
 	(segment
-		(start 116 48)
-		(end 116.901 47.099)
+		(start 119.77 56.633)
+		(end 119.77 57.695)
 		(width 0.5)
 		(layer "B.Cu")
@@
 	)
 	(segment
-		(start 117.23 57.695)
-		(end 117.23 55.945)
+		(start 122.690078 55.590078)
+		(end 120.812922 55.590078)
 		(width 0.5)
 		(layer "B.Cu")
@@
 	)
 	(segment
-		(start 134.036 48.25)
-		(end 132.885 47.099)
+		(start 128.956 49.324156)
+		(end 122.690078 55.590078)
 		(width 0.5)
 		(layer "B.Cu")
