File: KiCAD/projet-capteur/projet-capteur.kicad_sch (KiCad schematic)
At the start: 21 parts, among them J1 Power, J2 Analog, J3 Digital/PWM, J4 Digital/PWM, U2 LTC1050

Commit message: Beautification du Schematique
Connections:
- net *10 renamed CS Pot
- net *11 renamed SDI Pot
- net *9 renamed DATA Serv
- net 13 renamed SCK Pot
Other:
- note added: "ARDUINO UNO"
- note added: "BLUETOOTH"
- note added: "DIGITAL POTENTIOMETER"
- note added: "FLEX SENSOR"
- note added: "GRAPHITE SENSOR"
- note added: "OLED"
- note added: "ROTARY ENCODER"
- note added: "SERVO MOTOR"
- note added: "TRANSIMPEDANCE AMPLIFIER"
- title: (none) -> Projet Capteur - Graphite Sensor
- moved on the sheet: C4, CG1, FS1, J1, J2, J3, J4, MCP1, R6, ROE1, S1, U1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
